File: ESP32Pet PCB/ESP32Pet.kicad_sch (KiCad schematic)
At the start: 0 parts

Commit message: Schematic Updated
Other:
- sheet macros renamed macros + mounting holes + fudicials
- sheet microcontroller renamed ESP-32-WROOM
- removed sheet Battery Percent Logic
- removed sheet OnOff Logic
Changed lines of the file:
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@@
 	(paper "A4")
-	(sheet
-		(at 111.76 95.25)
-		(size 49.53 29.21)
-		(exclude_from_sim no)
-		(in_bom yes)
-		(on_board yes)
-		(dnp no)
-		(fields_autoplaced yes)
-		(stroke
-			(width 0.1524)
-			(type solid)
-		)
-		(fill
-			(color 0 0 0 0.0000)
-		)
-		(property "Sheetname" "OnOff Logic"
-			(at 111.76 94.5384 0)
-			(effects
-				(font
-					(size 1.27 1.27)
-				)
-				(justify left bottom)
-			)
-		)
-		(property "Sheetfile" "off_off_logic.kicad_sch"
-			(at 111.76 125.0446 0)
-			(effects
-				(font
-					(size 1.27 1.27)
-				)
-				(justify left top)
-			)
-		)
-		(instances
-			(project "ESP32Pet"
-				(path "/397abc7c-300b-4d6f-9337-33290484b5ae"
-					(page "6")
-				)
-			)
-		)
-	)
 	(sheet
 		(at 167.64 52.07)
@@
 			(color 0 0 0 0.0000)
 		)
-		(property "Sheetname" "macros"
+		(property "Sheetname" "macros + mounting holes + fudicials"
 			(at 167.64 51.3584 0)
 			(effects
@@
 	)
 	(sheet
-		(at 52.07 95.25)
+		(at 110.49 92.71)
 		(size 50.8 29.21)
 		(exclude_from_sim no)
@@
 		)
 		(property "Sheetname" "Power"
-			(at 52.07 94.5384 0)
+			(at 110.49 91.9984 0)
 			(effects
 				(font
@@
 		)
 		(property "Sheetfile" "power.kicad_sch"
-			(at 52.07 125.0446 0)
+			(at 110.49 122.5046 0)
 			(effects
 				(font
@@
 				(path "/397abc7c-300b-4d6f-9337-33290484b5ae"
 					(page "5")
-				)
-			)
-		)
-	)
-	(sheet
-		(at 170.18 95.25)
-		(size 50.8 30.48)
-		(exclude_from_sim no)
-		(in_bom yes)
-		(on_board yes)
-		(dnp no)
-		(fields_autoplaced yes)
-		(stroke
-			(width 0.1524)
-			(type solid)
-		)
-		(fill
-			(color 0 0 0 0.0000)
-		)
-		(property "Sheetname" "Battery Percent Logic"
-			(at 170.18 94.5384 0)
-			(effects
-				(font
-					(size 1.27 1.27)
-				)
-				(justify left bottom)
-			)
-		)
-		(property "Sheetfile" "battery_logic.kicad_sch"
-			(at 170.18 126.3146 0)
-			(effects
-				(font
-					(size 1.27 1.27)
-				)
-				(justify left top)
-			)
-		)
-		(instances
-			(project "ESP32Pet"
-				(path "/397abc7c-300b-4d6f-9337-33290484b5ae"
-					(page "7")
 				)
 			)
@@
 			(color 0 0 0 0.0000)
 		)
-		(property "Sheetname" "microcontroller"
+		(property "Sheetname" "ESP-32-WROOM"
 			(at 52.07 51.3584 0)
 			(effects
