File: ESP32Pet PCB/tft_lcd.kicad_sch (KiCad schematic)
At the start: 0 parts

Commit message: Schematic Updated
Parts:
- added U4: TFT LCD, ST7735:TFT LCD 1.8inch 128x160 w_ SD Card Slot, symbol ST7735 TFT:TFT LCD
Connections:
- new net 3.3V: U4. (CS)
- new net GND: U4. (CS)
- new net TFT_CLK: U4. (CS)
- new net TFT_CS: U4. (CS)
- new net TFT_RESET: U4. (CS)
- new net TFT_RS: U4. (CS)
- new net TFT_SDA: U4. (CS)

Commit message: Schematic complete, created custom footprints and symbols for TFT LCD
Parts:
- removed U4: TFT LCD, ST7735:TFT LCD 1.8inch 128x160 w_ SD Card Slot, symbol ST7735 TFT:TFT LCD
- added U2: TFT LCD, symbol ST7735 TFT:TFT LCD
Connections:
- net 3.3V: now also U2.1 (VCC)
- net GND: now also U2.2 (GND1), U2.3 (GND2)
- net TFT_CLK: now also U2.4 (CLK)
- net TFT_CS: now also U2.8 (CS)
- net TFT_RESET: now also U2.7 (RST)
- net TFT_RS: now also U2.6 (RS)
- net TFT_SDA: now also U2.5 (SDA)
Changed lines of the file:
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@@
+		)
+	)
+	(global_label "TFT_RESET"
+		(shape input)
+		(at 168.91 96.52 180)
+		(fields_autoplaced yes)
+		(effects
+			(font
+				(size 1.27 1.27)
+			)
+			(justify right)
+		)
+		(property "Intersheetrefs" "${INTERSHEET_REFS}"
+			(at 156.1883 96.52 0)
+			(effects
+				(font
+					(size 1.27 1.27)
+				)
+				(justify right)
+				(hide yes)
+			)
 		)
 	)
@@
 		)
 	)
-	(global_label "TFT_RESET"
-		(shape input)
-		(at 168.91 96.52 180)
-		(fields_autoplaced yes)
-		(effects
-			(font
-				(size 1.27 1.27)
-			)
-			(justify right)
-		)
-		(property "Intersheetrefs" "${INTERSHEET_REFS}"
-			(at 156.1883 96.52 0)
-			(effects
-				(font
-					(size 1.27 1.27)
-				)
-				(justify right)
-				(hide yes)
-			)
-		)
-	)
 	(global_label "TFT_CLK"
 		(shape input)
@@
 				(justify right)
 				(hide yes)
+			)
+		)
+	)
+	(symbol
+		(lib_id "power:GND")
+		(at 152.4 80.01 0)
+		(unit 1)
+		(exclude_from_sim no)
+		(in_bom yes)
+		(on_board yes)
+		(dnp no)
+		(fields_autoplaced yes)
+		(property "Reference" "#PWR02"
+			(at 152.4 86.36 0)
+			(effects
+				(font
+					(size 1.27 1.27)
+				)
+				(hide yes)
+			)
+		)
+		(property "Value" "GND"
+			(at 152.4 85.09 0)
+			(effects
+				(font
+					(size 1.27 1.27)
+				)
+			)
+		)
+		(property "Footprint" ""
+			(at 152.4 80.01 0)
+			(effects
+				(font
+					(size 1.27 1.27)
+				)
+				(hide yes)
+			)
+		)
+		(property "Datasheet" ""
+			(at 152.4 80.01 0)
+			(effects
+				(font
+					(size 1.27 1.27)
+				)
+				(hide yes)
+			)
+		)
+		(property "Description" "Power symbol creates a global label with name \"GND\" , ground"
+			(at 152.4 80.01 0)
+			(effects
+				(font
+					(size 1.27 1.27)
+				)
+				(hide yes)
+			)
+		)
+		(pin "1"
+		)
+		(instances
+			(project ""
+				(path "/397abc7c-300b-4d6f-9337-33290484b5ae/6de349e7-ced3-4959-8be3-0b8312a7c7a3"
+					(reference "#PWR02")
+					(unit 1)
+				)
 			)
 		)
@@
 		(dnp no)
 		(fields_autoplaced yes)
-		(property "Reference" "U4"
-			(at 175.9585 67.31 0)
-			(effects
-				(font
-					(size 1.27 1.27)
-				)
+		(property "Reference" "U2"
+			(at 184.15 86.3599 0)
+			(effects
+				(font
+					(size 1.27 1.27)
+				)
+				(justify left)
 			)
 		)
 		(property "Value" "TFT LCD"
-			(at 175.9585 69.85 0)
-			(effects
-				(font
-					(size 1.27 1.27)
-				)
-			)
-		)
-		(property "Footprint" "ST7735:TFT LCD 1.8inch 128x160 w_ SD Card Slot"
+			(at 184.15 88.8999 0)
+			(effects
+				(font
+					(size 1.27 1.27)
+				)
+				(justify left)
+			)
+		)
+		(property "Footprint" ""
 			(at 144.78 110.236 0)
 			(do_not_autoplace yes)
@@
 			)
 		)
-		(pin ""
-		)
-		(pin ""
-		)
-		(pin ""
-		)
-		(pin ""
-		)
-		(pin ""
-		)
-		(pin ""
-		)
-		(pin ""
-		)
-		(pin ""
+		(pin "2"
+		)
+		(pin "4"
+		)
+		(pin "5"
+		)
+		(pin "6"
+		)
+		(pin "7"
+		)
+		(pin "3"
+		)
+		(pin "8"
+		)
+		(pin "1"
 		)
 		(instances
 			(project ""
 				(path "/397abc7c-300b-4d6f-9337-33290484b5ae/6de349e7-ced3-4959-8be3-0b8312a7c7a3"
-					(reference "U4")
+					(reference "U2")
 					(unit 1)
 				)
-			)
-		)
-	)
-	(symbol
-		(lib_id "power:GND")
-		(at 152.4 80.01 0)
-		(unit 1)
-		(exclude_from_sim no)
-		(in_bom yes)
-		(on_board yes)
-		(dnp no)
-		(fields_autoplaced yes)
-		(property "Reference" "#PWR02"
-			(at 152.4 86.36 0)
-			(effects
-				(font
-					(size 1.27 1.27)
-				)
-				(hide yes)
-			)
-		)
-		(property "Value" "GND"
-			(at 152.4 85.09 0)
-			(effects
-				(font
-					(size 1.27 1.27)
-				)
-			)
-		)
-		(property "Footprint" ""
-			(at 152.4 80.01 0)
-			(effects
-				(font
-					(size 1.27 1.27)
-				)
-				(hide yes)
-			)
-		)
-		(property "Datasheet" ""
-			(at 152.4 80.01 0)
-			(effects
-				(font
-					(size 1.27 1.27)
-				)
-				(hide yes)
-			)
-		)
-		(property "Description" "Power symbol creates a global label with name \"GND\" , ground"
-			(at 152.4 80.01 0)
-			(effects
-				(font
-					(size 1.27 1.27)
-				)
-				(hide yes)
-			)
-		)
-		(pin "1"
-		)
-		(instances
-			(project ""
-				(path "/397abc7c-300b-4d6f-9337-33290484b5ae/6de349e7-ced3-4959-8be3-0b8312a7c7a3"
-					(reference "#PWR02")
-					(unit 1)
-				)

Commit message: PCB Design Complete
Parts:
- U2: footprint (none) -> ST7735:TFT LCD 1.8inch 128x160 w_ SD Card Slot
Changed lines of the file:
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@@
 			)
 		)
-		(property "Footprint" ""
+		(property "Footprint" "ST7735:TFT LCD 1.8inch 128x160 w_ SD Card Slot"
 			(at 144.78 110.236 0)
 			(do_not_autoplace yes)
